Commit message: updating code

File: sgrobot/description/sg_description_27_march.urdf.xacro (robot description, xacro)
@@ -5,4 +5,16 @@
 <!-- =================================================================================== -->
 <robot name="SG_robot" xmlns:xacro="http://www.ros.org/wiki/xacro">
+    <!--<gazebo>
+       <plugin name="gazebo_ros_control" filename="libgazebo_ros_control.so">
+       <robotNamespace>/SG_robot</robotNamespace>
+       </plugin>
+ </gazebo> -->
+    <gazebo>
+        <plugin filename="libgazebo_ros_control.so" name="gazebo_ros_control">
+            <robotNamespace>/SG_robot</robotNamespace>
+            <robotSimType>gazebo_ros_control/DefaultRobotHWSim</robotSimType>
+            <legacyModeNS>true</legacyModeNS>
+        </plugin>
+    </gazebo>
     <link name="world">
         <visual>
@@ -235,5 +247,5 @@
         <child link="gripper_right_link" />
         <axis xyz="0 1 0" />
-        <limit effort="1.5" lower="0.0" upper="0.03" velocity="6.178465545" />
+        <limit effort="1.5" lower="0.03" upper="0.0" velocity="6.178465545" />
     </joint>
     <link name="gripper_right_link">
@@ -290,8 +302,8 @@
         <type>transmission_interface/SimpleTransmission</type>
         <joint name="shoulder_yaw_joint">
-            <hardwareInterface>PositionJointInterface</hardwareInterface>
+            <hardwareInterface>hardware_interface/EffortJointInterface</hardwareInterface>
         </joint>
         <actuator name="shoulder_yaw_motor">
-            <hardwareInterface>PositionJointInterface</hardwareInterface>
+            <hardwareInterface>hardware_interface/EffortJointInterface</hardwareInterface>
             <mechanicalReduction>1</mechanicalReduction>
         </actuator>
@@ -300,8 +312,8 @@
         <type>transmission_interface/SimpleTransmission</type>
         <joint name="shoulder_pitch_joint">
-            <hardwareInterface>PositionJointInterface</hardwareInterface>
+            <hardwareInterface>hardware_interface/EffortJointInterface</hardwareInterface>
         </joint>
         <actuator name="shoulder_pitch_motor">
-            <hardwareInterface>PositionJointInterface</hardwareInterface>
+            <hardwareInterface>hardware_interface/EffortJointInterface</hardwareInterface>
             <mechanicalReduction>1</mechanicalReduction>
         </actuator>
@@ -310,8 +322,8 @@
         <type>transmission_interface/SimpleTransmission</type>
         <joint name="elbow_pitch_joint">
-            <hardwareInterface>PositionJointInterface</hardwareInterface>
+            <hardwareInterface>hardware_interface/EffortJointInterface</hardwareInterface>
         </joint>
         <actuator name="elbow_pitch_motor">
-            <hardwareInterface>PositionJointInterface</hardwareInterface>
+            <hardwareInterface>hardware_interface/EffortJointInterface</hardwareInterface>
             <mechanicalReduction>1</mechanicalReduction>
         </actuator>
@@ -320,8 +332,8 @@
         <type>transmission_interface/SimpleTransmission</type>
         <joint name="wrist_pitch_joint">
-            <hardwareInterface>PositionJointInterface</hardwareInterface>
+            <hardwareInterface>hardware_interface/EffortJointInterface</hardwareInterface>
         </joint>
         <actuator name="wrist_pitch_motor">
-            <hardwareInterface>PositionJointInterface</hardwareInterface>
+            <hardwareInterface>hardware_interface/EffortJointInterface</hardwareInterface>
             <mechanicalReduction>1</mechanicalReduction>
         </actuator>
@@ -330,26 +342,10 @@
         <type>transmission_interface/SimpleTransmission</type>
         <joint name="wrist_roll_joint">
-            <hardwareInterface>PositionJointInterface</hardwareInterface>
+            <hardwareInterface>hardware_interface/EffortJointInterface</hardwareInterface>
         </joint>
         <actuator name="wrist_roll_motor">
-            <hardwareInterface>PositionJointInterface</hardwareInterface>
-            <mechanicalReduction>1</mechanicalReduction>
-        </actuator>
-    </transmission>
-    <transmission name="gripper_revolute_trans">
-        <type>transmission_interface/SimpleTransmission</type>
-        <joint name="gripper_right_joint">
-            <hardwareInterface>PositionJointInterface</hardwareInterface>
-        </joint>
-        <actuator name="gripper_right_motor">
-            <hardwareInterface>PositionJointInterface</hardwareInterface>
-            <mechanicalReduction>1</mechanicalReduction>
-        </actuator>
-    </transmission>
-     <gazebo>
-    <plugin name="gazebo_ros_control" filename="libgazebo_ros_control.so">
-      <robotNamespace>/SG_robot</robotNamespace>
-      <legacyModeNS>true</legacyModeNS>
-    </plugin>
-  </gazebo>
+            <hardwareInterface>hardware_interface/EffortJointInterface</hardwareInterface>
+            <mechanicalReduction>1</mechanicalReduction>
+        </actuator>
+    </transmission>
 </robot>

File: sgrobot/description/sg_description_original.urdf.xacro (robot description, xacro)
@@ -48,5 +48,5 @@
         <child link="shoulder_link" />
         <axis xyz="0 0 1" />
-        <limit effort="1.5" lower="-3.141593" upper="3.141593" velocity="6.178465545" />
+        <limit effort="1.0" lower="-3.141593" upper="3.141593" velocity="6.178465545" />
     </joint>
     <link name="shoulder_link">
@@ -78,5 +78,5 @@
         <child link="bicep_link" />
         <axis xyz="0 0 -1" />
-        <limit effort="3.0" lower="-1.5707965" upper="1.5707965" velocity="6.178465545" />
+        <limit effort="1.0" lower="-1.5707965" upper="1.5707965" velocity="6.178465545" />
     </joint>
     <link name="bicep_link">
@@ -108,5 +108,5 @@
         <child link="forearm_link" />
         <axis xyz="0 1 0" />
-        <limit effort="3.0" lower="-1.5707965" upper="1.5707965" velocity="6.178465545" />
+        <limit effort="1.0" lower="-1.5707965" upper="1.5707965" velocity="6.178465545" />
     </joint>
     <link name="forearm_link">
@@ -138,5 +138,5 @@
         <child link="wrist_1_link" />
         <axis xyz="0 1 0" />
-        <limit effort="1.5" lower="-1.7" upper="1.9" velocity="6.178465545" />
+        <limit effort="1.0" lower="-1.7" upper="1.9" velocity="6.178465545" />
     </joint>
     <link name="wrist_1_link">
@@ -168,5 +168,5 @@
         <child link="wrist_2_link" />
         <axis xyz="1 0 0" />
-        <limit effort="1.5" lower="-3.141593" upper="3.141593" velocity="6.178465545" />
+        <limit effort="1.0" lower="-3.141593" upper="3.141593" velocity="6.178465545" />
     </joint>
     <link name="wrist_2_link">
@@ -198,5 +198,5 @@
         <child link="gripper_guide_link" />
         <axis xyz="0 0 1" />
-        <limit effort="1.5" lower="0" upper="1.57" velocity="6.178465545" />
+        <limit effort="1.0" lower="0" upper="1.57" velocity="6.178465545" />
     </joint>
     <link name="gripper_guide_link">
@@ -227,5 +227,5 @@
         <child link="gripper_aux_link" />
         <axis xyz="0 0 1" />
-        <limit effort="0" lower="-3.141593" upper="3.141593" velocity="0.5" />
+        <limit effort="1.0" lower="-3.141593" upper="3.141593" velocity="0.5" />
     </joint>
     <link name="gripper_aux_link" />
@@ -263,5 +263,5 @@
         <child link="gripper_left_link" />
         <axis xyz="0 1 0" />
-        <limit effort="1.5" lower="-1.9" upper="0" velocity="6.178465545" />
+        <limit effort="1.0" lower="-1.9" upper="0" velocity="6.178465545" />
         <mimic joint="gripper_right_joint" multiplier="-1.0" />
     </joint>
@@ -290,9 +290,9 @@
         <type>transmission_interface/SimpleTransmission</type>
         <joint name="shoulder_yaw_joint">
-            <hardwareInterface>PositionJointInterface</hardwareInterface>
+            <hardwareInterface>hardware_interface/EffortJointInterface</hardwareInterface>
         </joint>
         <actuator name="shoulder_yaw_motor">
-            <hardwareInterface>PositionJointInterface</hardwareInterface>
-            <mechanicalReduction>1</mechanicalReduction>
+            <hardwareInterface>EffortJointInterface</hardwareInterface>
+            <mechanicalReduction>150</mechanicalReduction>
         </actuator>
     </transmission>
@@ -300,9 +300,9 @@
         <type>transmission_interface/SimpleTransmission</type>
         <joint name="shoulder_pitch_joint">
-            <hardwareInterface>PositionJointInterface</hardwareInterface>
+            <hardwareInterface>hardware_interface/EffortJointInterface</hardwareInterface>
         </joint>
         <actuator name="shoulder_pitch_motor">
-            <hardwareInterface>PositionJointInterface</hardwareInterface>
-            <mechanicalReduction>1</mechanicalReduction>
+            <hardwareInterface>EffortJointInterface</hardwareInterface>
+            <mechanicalReduction>100</mechanicalReduction>
         </actuator>
     </transmission>
@@ -310,9 +310,9 @@
         <type>transmission_interface/SimpleTransmission</type>
         <joint name="elbow_pitch_joint">
-            <hardwareInterface>PositionJointInterface</hardwareInterface>
+            <hardwareInterface>hardware_interface/EffortJointInterface</hardwareInterface>
         </joint>
         <actuator name="elbow_pitch_motor">
-            <hardwareInterface>PositionJointInterface</hardwareInterface>
-            <mechanicalReduction>1</mechanicalReduction>
+            <hardwareInterface>EffortJointInterface</hardwareInterface>
+            <mechanicalReduction>100</mechanicalReduction>
         </actuator>
     </transmission>
@@ -320,9 +320,9 @@
         <type>transmission_interface/SimpleTransmission</type>
         <joint name="wrist_pitch_joint">
-            <hardwareInterface>PositionJointInterface</hardwareInterface>
+            <hardwareInterface>hardware_interface/EffortJointInterface</hardwareInterface>
         </joint>
         <actuator name="wrist_pitch_motor">
-            <hardwareInterface>PositionJointInterface</hardwareInterface>
-            <mechanicalReduction>1</mechanicalReduction>
+            <hardwareInterface>EffortJointInterface</hardwareInterface>
+            <mechanicalReduction>200</mechanicalReduction>
         </actuator>
     </transmission>
@@ -330,9 +330,9 @@
         <type>transmission_interface/SimpleTransmission</type>
         <joint name="wrist_roll_joint">
-            <hardwareInterface>PositionJointInterface</hardwareInterface>
+            <hardwareInterface>hardware_interface/EffortJointInterface</hardwareInterface>
         </joint>
         <actuator name="wrist_roll_motor">
-            <hardwareInterface>PositionJointInterface</hardwareInterface>
-            <mechanicalReduction>1</mechanicalReduction>
+            <hardwareInterface>EffortJointInterface</hardwareInterface>
+            <mechanicalReduction>100</mechanicalReduction>
         </actuator>
     </transmission>
@@ -340,9 +340,9 @@
         <type>transmission_interface/SimpleTransmission</type>
         <joint name="gripper_right_joint">
-            <hardwareInterface>PositionJointInterface</hardwareInterface>
+            <hardwareInterface>hardware_interface/EffortJointInterface</hardwareInterface>
         </joint>
         <actuator name="gripper_right_motor">
-            <hardwareInterface>PositionJointInterface</hardwareInterface>
-            <mechanicalReduction>1</mechanicalReduction>
+            <hardwareInterface>EffortJointInterface</hardwareInterface>
+            <mechanicalReduction>100</mechanicalReduction>
         </actuator>
     </transmission>
@@ -350,4 +350,5 @@
     <plugin name="gazebo_ros_control" filename="libgazebo_ros_control.so">
       <robotNamespace>/SG_robot</robotNamespace>
+      <!--<robotSimType>gazebo_ros_control/DefaultRobotHWSim</robotSimType>-->
       <legacyModeNS>true</legacyModeNS>
     </plugin>
